File: schematics/mcu.kicad_sch (KiCad schematic)
At the start: 3 parts, among them SW1 SW_ESP_ EN, U1 ESP32-PICO-MINI-02

Commit message: Plot revision 1 - partial submission
Connections:
- net TWAI_BUS_ON_OFF: no longer names the net of U1.27 (IO7)
- net TWAI_CLK_OUT: no longer names the net of U1.28 (IO8)
- no-connect marks 13 -> 15
Changed lines of the file:
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@@
+	)
+	(no_connect
+		(at 129.54 69.85)
 	)
 	(no_connect
@@
 	(no_connect
 		(at 160.02 77.47)
+	)
+	(no_connect
+		(at 129.54 67.31)
 	)
 	(no_connect
@@
 	(wire
 		(pts
-			(xy 120.65 69.85) (xy 129.54 69.85)
-		)
-		(stroke
-			(width 0)
-			(type default)
-		)
-	)
-	(wire
-		(pts
 			(xy 160.02 148.59) (xy 170.18 148.59)
 		)
@@
 		(pts
 			(xy 160.02 133.35) (xy 170.18 133.35)
-		)
-		(stroke
-			(width 0)
-			(type default)
-		)
-	)
-	(wire
-		(pts
-			(xy 120.65 67.31) (xy 129.54 67.31)
 		)
 		(stroke
@@
 		)
 	)
-	(hierarchical_label "TWAI_CLK_OUT"
-		(shape output)
-		(at 120.65 69.85 180)
-		(effects
-			(font
-				(size 1.27 1.27)
-			)
-			(justify right)
-		)
-	)
 	(hierarchical_label "ISL_DE"
 		(shape output)
@@
 		(effects
 			(font
-				(size 1.27 1.27)
-			)
-			(justify right)
-		)
-	)
-	(hierarchical_label "TWAI_BUS_ON_OFF"
-		(shape bidirectional)
-		(at 120.65 67.31 180)
-		(effects
-			(font
