File: schematics/programmer_and_debugger.kicad_sch (KiCad schematic)
At the start: 4 parts, among them J1 USB_C_Receptacle_USB2.0_16P, U3 FT232RL

Commit message: Plot revision 1 - partial submission
Parts:
- added C16: 0.1uF, Capacitor_THT:C_Disc_D3.4mm_W2.1mm_P2.50mm, symbol Device:C_Small
Connections:
- net GND: now also C16.2
- net VCC: now also C16.1
- net VBUS: no longer names the net of J1.A4 (VBUS), J1.A9 (VBUS), J1.B4 (VBUS), J1.B9 (VBUS)
- no-connect marks 16 -> 19
Changed lines of the file:
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@@
+	)
+	(junction
+		(at 181.61 54.61)
+		(diameter 0)
+		(color 0 0 0 0)
 	)
 	(junction
@@
 	)
 	(no_connect
+		(at 158.75 87.63)
+	)
+	(no_connect
 		(at 199.39 102.87)
 	)
@@
 	)
 	(no_connect
+		(at 111.76 71.12)
+	)
+	(no_connect
 		(at 199.39 95.25)
 	)
@@
 	)
 	(no_connect
+		(at 158.75 69.85)
+	)
+	(no_connect
 		(at 199.39 100.33)
 	)
@@
 	(wire
 		(pts
+			(xy 181.61 54.61) (xy 181.61 57.15)
+		)
+		(stroke
+			(width 0)
+			(type default)
+		)
+	)
+	(wire
+		(pts
 			(xy 181.61 57.15) (xy 181.61 62.23)
 		)
@@
 	(wire
 		(pts
+			(xy 209.55 55.88) (xy 209.55 54.61)
+		)
+		(stroke
+			(width 0)
+			(type default)
+		)
+	)
+	(wire
+		(pts
 			(xy 88.9 111.76) (xy 96.52 111.76)
 		)
@@
 	(wire
 		(pts
+			(xy 209.55 54.61) (xy 181.61 54.61)
+		)
+		(stroke
+			(width 0)
+			(type default)
+		)
+	)
+	(wire
+		(pts
 			(xy 179.07 113.03) (xy 179.07 116.84)
 		)
@@
 	(wire
 		(pts
+			(xy 209.55 60.96) (xy 209.55 63.5)
+		)
+		(stroke
+			(width 0)
+			(type default)
+		)
+	)
+	(wire
+		(pts
 			(xy 96.52 109.22) (xy 96.52 111.76)
 		)
@@
 	(wire
 		(pts
-			(xy 181.61 52.07) (xy 181.61 57.15)
+			(xy 181.61 52.07) (xy 181.61 54.61)
 		)
 		(stroke
@@
 			)
 			(justify right bottom)
+		)
+	)
+	(hierarchical_label "GND"
+		(shape input)
+		(at 209.55 63.5 270)
+		(effects
+			(font
+				(size 1.27 1.27)
+			)
+			(justify right)
 		)
 	)
@@
 		)
 	)
-	(hierarchical_label "VBUS"
-		(shape input)
-		(at 111.76 71.12 0)
+	(hierarchical_label "VCC"
+		(shape input)
+		(at 181.61 52.07 90)
 		(effects
 			(font
@@
 		)
 	)
-	(hierarchical_label "VCC"
-		(shape input)
-		(at 181.61 52.07 90)
+	(hierarchical_label "RXD"
+		(shape input)
+		(at 199.39 72.39 0)
 		(effects
 			(font
@@
 		)
 	)
-	(hierarchical_label "RXD"
-		(shape input)
-		(at 199.39 72.39 0)
-		(effects
-			(font
-				(size 1.27 1.27)
-			)
-			(justify left)
-		)
-	)
 	(hierarchical_label "GND"
 		(shape input)
@@
 		)
 	)
+	(symbol
+		(lib_id "Device:C_Small")
+		(at 209.55 58.42 0)
+		(mirror y)
+		(unit 1)
+		(body_style 1)
+		(exclude_from_sim no)
+		(in_bom yes)
+		(on_board yes)
+		(in_pos_files yes)
+		(dnp no)
+		(fields_autoplaced yes)
+		(property "Reference" "C16"
+			(at 207.01 57.1562 0)
+			(show_name no)
+			(do_not_autoplace no)
+			(effects
+				(font
+					(size 1.27 1.27)
+				)
+				(justify left)
+			)
+		)
+		(property "Value" "0.1uF"
+			(at 207.01 59.6962 0)
+			(show_name no)
+			(do_not_autoplace no)
+			(effects
+				(font
+					(size 1.27 1.27)
+				)
+				(justify left)
+			)
+		)
+		(property "Footprint" "Capacitor_THT:C_Disc_D3.4mm_W2.1mm_P2.50mm"
+			(at 209.55 58.42 0)
+			(hide yes)
+			(show_name no)
+			(do_not_autoplace no)
+			(effects
+				(font
+					(size 1.27 1.27)
+				)
+			)
+		)
+		(property "Datasheet" ""
+			(at 209.55 58.42 0)
+			(hide yes)
+			(show_name no)
+			(do_not_autoplace no)
+			(effects
+				(font
+					(size 1.27 1.27)
+				)
+			)
+		)
+		(property "Description" "Unpolarized capacitor, small symbol"
+			(at 209.55 58.42 0)
+			(hide yes)
+			(show_name no)
+			(do_not_autoplace no)
+			(effects
+				(font
+					(size 1.27 1.27)
+				)
+			)
+		)
+		(pin "1"
+		)
+		(pin "2"
+		)
+		(instances
+			(project "sensor_node_custom_board"
+				(path "/71a54788-2d41-499b-94da-7868bc933cd8/7ef40683-6994-4b58-892d-20d1e88778d4"
+					(reference "C16")
+					(unit 1)
+				)
+			)
+		)
+	)
