File: schematics/sensor_node_custom_board.kicad_pcb (KiCad board)
At the start: 2 copper layers, 243.5 x 159.5 mm, 57 parts, among them J1 USB_C_Receptacle_USB2.0_16P, J10 RTD3, J11 RTD4, J12 RTD5, J13 RTD7, J14 RTD6, J15 RTD8, J16 RTD9, J17 RTD10, J18 RTD11, J19 RTD12, J20 RTD13, J21 RTD14, J22 RTD15, J23 RTD16, J24 RTD_B (Breakout), J25 RTD_A, J26 RTD_B, J27 CAN, J3 Screw_Terminal_01x03, J6 RTD_A (Breakout), J7 MODBUS RTU, J8 RTD1, J9 RTD2, SW1 SW_ESP_ EN, SW2 SW_Nidec_CAS-120A1, U1 ESP32-PICO-MINI-02, U11 ISL3175E, U2 XL1509-5.0, U3 FT232RL, U4 XL1509-3.3, U5 MAX31865xTP, U6 CD74HC4067M, U7 CD74HC4067M, U8 CD74HC4067M, U9 SN65HVD255D

Commit message: Plot revision 1 - partial submission
Parts:
- added C15: 0.1uF, Capacitor_THT:C_Disc_D3.4mm_W2.1mm_P2.50mm, F.Cu at (178.6, 113.8)
- added C16: 0.1uF, Capacitor_THT:C_Disc_D3.4mm_W2.1mm_P2.50mm, F.Cu at (178.6, 119.5)
- moved C2 53.3 mm to (257.0, 50.0)
- moved C1 32.4 mm to (229.5, 82.5)
- moved C3 6.66 mm to (207.5, 61.5)
Connections:
- J1 pad A4: Net-(J1-VBUS-PadA4) -> unconnected-(J1-VBUS-PadA4)_3
- J1 pad A9: Net-(J1-VBUS-PadA4) -> unconnected-(J1-VBUS-PadA4)_1
- J1 pad B4: Net-(J1-VBUS-PadA4) -> unconnected-(J1-VBUS-PadA4)_2
- J1 pad B9: Net-(J1-VBUS-PadA4) -> unconnected-(J1-VBUS-PadA4)
- J27 pad 2: unconnected-(J27-Pad2) -> /Control Board/CAN Bus Controller/CANL
- J27 pad 3: /Control Board/CAN Bus Controller/CANH -> /Control Board/Power Supply/COM_GND
- J27 pad 7: unconnected-(J27-Pad7) -> /Control Board/CAN Bus Controller/CANH
- J27 pad 8: /Control Board/CAN Bus Controller/CANL -> unconnected-(J27-Pad8)
- J27 pad 9: unconnected-(J27-Pad9) -> /Control Board/Power Supply/VBUS_3V3
- U1 pad 24: /Control Board/MCU/TWAI_RX -> /Control Board/TWAI_RX
- U1 pad 27: /Control Board/MCU/TWAI_BUS_ON_OFF -> unconnected-(U1-IO7-Pad27)
- U1 pad 28: /Control Board/MCU/TWAI_CLK_OUT -> unconnected-(U1-IO8-Pad28)
- U1 pad 29: /Control Board/MCU/TWAI_TX -> /Control Board/TWAI_TX
- U9 pad 1: /Control Board/CAN Bus Controller/TXD -> /Control Board/TWAI_TX
- U9 pad 2: /Control Board/CAN Bus Controller/GND -> /Control Board/Power Supply/COM_GND
- U9 pad 3: /Control Board/CAN Bus Controller/VCC -> /Control Board/Power Supply/VBUS_3V3
- U9 pad 4: /Control Board/CAN Bus Controller/RXD -> /Control Board/TWAI_RX
