File: schematics/sensor_node_custom_board.kicad_sch (KiCad schematic)
At the start: 0 parts

Commit message: Plot revision 1 - partial submission
Other:
- sheet MCU ports: added none; removed TWAI_BUS_ON_OFF, TWAI_CLK_OUT
- sheet Programmer & Debugger ports: added none; removed VCONN
Changed lines of the file:
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@@
+	(wire
+		(pts
+			(xy 189.23 53.34) (xy 185.42 53.34)
+		)
+		(stroke
+			(width 0)
+			(type default)
+		)
+	)
+	(wire
+		(pts
+			(xy 189.23 55.88) (xy 185.42 55.88)
+		)
+		(stroke
+			(width 0)
+			(type default)
+		)
+	)
 	(wire
 		(pts
@@
 	(wire
 		(pts
+			(xy 189.23 146.05) (xy 185.42 146.05)
+		)
+		(stroke
+			(width 0)
+			(type default)
+		)
+	)
+	(wire
+		(pts
 			(xy 189.23 106.68) (xy 185.42 106.68)
 		)
@@
 		(pts
 			(xy 189.23 78.74) (xy 185.42 78.74)
+		)
+		(stroke
+			(width 0)
+			(type default)
+		)
+	)
+	(wire
+		(pts
+			(xy 189.23 149.86) (xy 185.42 149.86)
 		)
 		(stroke
@@
 		)
 	)
+	(label "TWAI_TX"
+		(at 189.23 149.86 0)
+		(effects
+			(font
+				(size 1.27 1.27)
+			)
+			(justify left bottom)
+		)
+	)
+	(label "TWAI_RX"
+		(at 189.23 53.34 0)
+		(effects
+			(font
+				(size 1.27 1.27)
+			)
+			(justify left bottom)
+		)
+	)
 	(label "ESP_RXD0"
 		(at 189.23 20.32 0)
@@
 		)
 	)
+	(label "TWAI_RX"
+		(at 189.23 146.05 0)
+		(effects
+			(font
+				(size 1.27 1.27)
+			)
+			(justify left bottom)
+		)
+	)
 	(label "ESP_TXD0"
 		(at 189.23 106.68 0)
@@
 	(label "ISL_DE"
 		(at 189.23 43.18 0)
+		(effects
+			(font
+				(size 1.27 1.27)
+			)
+			(justify left bottom)
+		)
+	)
+	(label "TWAI_TX"
+		(at 189.23 55.88 0)
 		(effects
 			(font
@@
 			)
 		)
-		(pin "RXD" output
+		(pin "RXD" input
 			(at 185.42 146.05 0)
 			(effects
@@
 			)
 		)
-		(pin "TXD" input
+		(pin "TXD" output
 			(at 185.42 149.86 0)
 			(effects
@@
 			)
 		)
-		(pin "VCONN" bidirectional
-			(at 185.42 110.49 0)
-			(effects
-				(font
-					(size 1.27 1.27)
-				)
-				(justify right)
-			)
-		)
 		(instances
 			(project "sensor_node_custom_board"
@@
 			(effects
 				(font
-					(size 1.27 1.27)
-				)
-				(justify right)
-			)
-		)
-		(pin "TWAI_BUS_ON_OFF" bidirectional
-			(at 185.42 48.26 0)
-			(effects
-				(font
-					(size 1.27 1.27)
-				)
-				(justify right)
-			)
-		)
-		(pin "TWAI_CLK_OUT" output
-			(at 185.42 50.8 0)
-			(effects
-				(font
